File: ferry.kicad_pcb (KiCad board)
At the start: 2 copper layers, 130.2 x 122 mm, 42 parts

Commit message: Updated layout
Routing:
- net P18: track 141.8 -> 184.7 mm
Changed lines of the file:
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@@
   (segment (start 123.558796 88.210558) (end 123.933877 88.585639) (width 0.25) (layer "B.Cu") (net 5))
   (segment (start 191.229808 95.170192) (end 190.487495 95.170192) (width 0.25) (layer "F.Cu") (net 6))
+  (segment (start 130.71618 49.424112) (end 131.827373 50.535305) (width 0.25) (layer "F.Cu") (net 6))
   (segment (start 197.861019 77.261019) (end 197.861019 88.538981) (width 0.25) (layer "F.Cu") (net 6))
   (segment (start 195.862511 57.462511) (end 195.862511 71.937489) (width 0.25) (layer "F.Cu") (net 6))
@@
   (segment (start 142.16479 43.639013) (end 149.210855 36.592948) (width 0.25) (layer "F.Cu") (net 6))
   (segment (start 192.15 53.75) (end 195.862511 57.462511) (width 0.25) (layer "F.Cu") (net 6))
+  (segment (start 131.827373 59.123409) (end 128.551182 62.3996) (width 0.25) (layer "F.Cu") (net 6))
+  (segment (start 131.85918 43.639013) (end 130.71618 44.782013) (width 0.25) (layer "F.Cu") (net 6))
+  (segment (start 130.586721 64.435139) (end 130.586721 75.816651) (width 0.25) (layer "F.Cu") (net 6))
   (segment (start 168.006744 46.505289) (end 178.84389 46.505289) (width 0.25) (layer "F.Cu") (net 6))
   (segment (start 131.85918 43.639013) (end 142.16479 43.639013) (width 0.25) (layer "F.Cu") (net 6))
   (segment (start 197.861019 88.538981) (end 191.229808 95.170192) (width 0.25) (layer "F.Cu") (net 6))
+  (segment (start 130.71618 44.782013) (end 130.71618 49.424112) (width 0.25) (layer "F.Cu") (net 6))
+  (segment (start 131.827373 50.535305) (end 131.827373 59.123409) (width 0.25) (layer "F.Cu") (net 6))
   (segment (start 195.862511 71.937489) (end 195.784663 72.015337) (width 0.25) (layer "F.Cu") (net 6))
+  (segment (start 128.551182 62.3996) (end 130.586721 64.435139) (width 0.25) (layer "F.Cu") (net 6))
   (segment (start 178.84389 46.505289) (end 186.088601 53.75) (width 0.25) (layer "F.Cu") (net 6))
   (segment (start 186.088601 53.75) (end 192.15 53.75) (width 0.25) (layer "F.Cu") (net 6))
@@
   (segment (start 195.784663 72.015337) (end 195.784663 75.184663) (width 0.25) (layer "F.Cu") (net 6))
   (segment (start 158.094403 36.592948) (end 168.006744 46.505289) (width 0.25) (layer "F.Cu") (net 6))
+  (segment (start 130.586721 75.816651) (end 125.243184 81.160188) (width 0.25) (layer "F.Cu") (net 6))
   (segment (start 123.919985 79.836989) (end 125.243184 81.160188) (width 0.25) (layer "B.Cu") (net 6))
   (segment (start 124.354945 42.315814) (end 130.535981 42.315814) (width 0.25) (layer "B.Cu") (net 6))
